File: BILLEE_Science_Control_Module_V1/BILLEE_Science_Control_Module_V1.kicad_sch (KiCad schematic)
At the start: 0 parts

Commit message: Setup Schematic for kiddos
Other:
- removed sheet Teensy4.1
- added sheet Chemical Management System (cms.kicad_sch)
- added sheet Regolith Extraction Module (rem.kicad_sch)
- added sheet Sample Cache and Rotation System (scrs.kicad_sch)
- added sheet Science Control Module (scm.kicad_sch)
- added sheet UV Spectroscopy Module (uvs.kicad_sch)
- note added: "* Billee-RCM Flight Software Deployment"
- note added: "* Science Control Module Hardware Architecture"
- note added: "BILLEE Science Control Module"
- note added: "Resources:"
- note removed: "Block Diagram"
- company: (none) -> Bronco STAR
- title: (none) -> Science Control Module
