File: BILLEE_Science_Control_Module_V1/rem.kicad_sch (KiCad schematic)
At the start: 0 parts

Commit message: Updating Symbols and Setting up modules
Created symbols for the parts included in the Draw.io and included a preliminary outline
Parts:
- added M1: Motor_Servo, symbol Motor:Motor_Servo
- added SW1, SW2, SW3, SW4, SW5, SW6: SW_Nidec_CAS-120A1, Button_Switch_SMD:Nidec_Copal_CAS-120A, symbol Switch:SW_Nidec_CAS-120A1
- added U14, U15, U16, U17: (no value), symbol scm_lib:YellowJacket_5203
