File: BILLEE_Science_Control_Module_V1/scm.kicad_sch (KiCad schematic)
At the start: 0 parts

Commit message: Updating Symbols and Setting up modules
Created symbols for the parts included in the Draw.io and included a preliminary outline
Parts:
- added U1, U2: (no value), symbol scm_lib:Pololu Buck Converter
- added U10, U11, U12, U13, U7, U8, U9: (no value), symbol scm_lib:Teyleten_Relay
- added U3: (no value), symbol scm_lib:Anderson_Powerpole_Bulkhead
- added U4, U5: RoboClaw_2x7A, symbol scm_lib:Roboclaw2x7A
- added U6: PCA9685, 815:MODULE_815, symbol scm_lib:PCA9685
Connections:
- new net: U6.OE_1 (~{OE}), U6.OE_2 (~{OE})
- new net: U6.SCL_1 (SCL), U6.SCL_2 (SCL)
- new net: U6.SDA_1 (SDA), U6.SDA_2 (SDA)
- new net GND: U6.GND_1 (GND), U6.GND_10 (GND), U6.GND_11 (GND), U6.GND_12 (GND), U6.GND_13 (GND), U6.GND_14 (GND), U6.GND_15 (GND), U6.GND_16 (GND), U6.GND_17 (GND), U6.GND_18 (GND), U6.GND_2 (GND), U6.GND_3 (GND), U6.GND_4 (GND), U6.GND_5 (GND), U6.GND_6 (GND), U6.GND_7 (GND), U6.GND_8 (GND), U6.GND_9 (GND)
- new net V+: U6.V+_1 (V+), U6.V+_10 (V+), U6.V+_11 (V+), U6.V+_12 (V+), U6.V+_13 (V+), U6.V+_14 (V+), U6.V+_15 (V+), U6.V+_16 (V+), U6.V+_17 (V+), U6.V+_18 (V+), U6.V+_2 (V+), U6.V+_3 (V+), U6.V+_4 (V+), U6.V+_5 (V+), U6.V+_6 (V+), U6.V+_7 (V+), U6.V+_8 (V+), U6.V+_9 (V+)
- new net VCC: U6.VCC_1 (VCC), U6.VCC_2 (VCC)

Commit message: Added more components
last component that is missing is the pressure sensor amp but ki-cad crashed
Parts:
- added U67: (no value), symbol scm_lib:arducam_1080p_day_night_vision_usb_camera
- added YMH: (no value), symbol scm_lib:chemical_Pumps
Connections:
- no-connect marks 0 -> 1
Changed lines of the file:
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@@
 	(generator_version "10.0")
 	(paper "A4")
+	(no_connect
+		(at 175.26 90.17)
+	)
+	(symbol
+		(lib_id "scm_lib:chemical_Pumps")
+		(at 161.29 149.86 0)
+		(unit 1)
+		(body_style 1)
+		(exclude_from_sim no)
+		(in_bom yes)
+		(on_board yes)
+		(in_pos_files yes)
+		(dnp no)
+		(fields_autoplaced yes)
+		(property "Reference" "YMH"
+			(at 166.37 146.8119 0)
+			(show_name no)
+			(do_not_autoplace no)
+			(effects
+				(font
+					(size 1.27 1.27)
+				)
+				(justify left)
+			)
+		)
+		(property "Value" ""
+			(at 161.29 149.86 0)
+			(show_name no)
+			(do_not_autoplace no)
+			(effects
+				(font
+					(size 1.27 1.27)
+				)
+			)
+		)
+		(property "Footprint" ""
+			(at 161.29 149.86 0)
+			(hide yes)
+			(show_name no)
+			(do_not_autoplace no)
+			(effects
+				(font
+					(size 1.27 1.27)
+				)
+			)
+		)
+		(property "Datasheet" ""
+			(at 161.29 149.86 0)
+			(hide yes)
+			(show_name no)
+			(do_not_autoplace no)
+			(effects
+				(font
+					(size 1.27 1.27)
+				)
+			)
+		)
+		(property "Description" ""
+			(at 161.29 149.86 0)
+			(hide yes)
+			(show_name no)
+			(do_not_autoplace no)
+			(effects
+				(font
+					(size 1.27 1.27)
+				)
+			)
+		)
+		(pin "2"
+		)
+		(pin "1"
+		)
+		(instances
+			(project "BILLEE_Science_Control_Module_V1"
+				(path "/0ccdd54c-cb66-4dbe-ac7e-21982bafb0a6/431a2b87-8d6b-4f12-9148-b0247a47a425"
+					(reference "YMH")
+					(unit 1)
+				)
+			)
+		)
+	)
 	(symbol
 		(lib_id "scm_lib:Teyleten_Relay")
@@
 	)
 	(symbol
+		(lib_name "Roboclaw2x7A_1")
 		(lib_id "scm_lib:Roboclaw2x7A")
 		(at 68.58 80.01 0)
@@
 	)
 	(symbol
+		(lib_id "scm_lib:arducam_1080p_day_night_vision_usb_camera")
+		(at 160.02 130.81 270)
+		(unit 1)
+		(body_style 1)
+		(exclude_from_sim no)
+		(in_bom yes)
+		(on_board yes)
+		(in_pos_files yes)
+		(dnp no)
+		(property "Reference" "U67"
+			(at 167.64 130.81 90)
+			(show_name no)
+			(do_not_autoplace no)
+			(effects
+				(font
+					(size 1.27 1.27)
+				)
+				(justify left)
+			)
+		)
+		(property "Value" ""
+			(at 160.02 130.81 0)
+			(show_name no)
+			(do_not_autoplace no)
+			(effects
+				(font
+					(size 1.27 1.27)
+				)
+			)
+		)
+		(property "Footprint" ""
+			(at 160.02 130.81 0)
+			(hide yes)
+			(show_name no)
+			(do_not_autoplace no)
+			(effects
+				(font
+					(size 1.27 1.27)
+				)
+			)
+		)
+		(property "Datasheet" ""
+			(at 160.02 130.81 0)
+			(hide yes)
+			(show_name no)
+			(do_not_autoplace no)
+			(effects
+				(font
+					(size 1.27 1.27)
+				)
+			)
+		)
+		(property "Description" ""
+			(at 160.02 130.81 0)
+			(hide yes)
+			(show_name no)
+			(do_not_autoplace no)
+			(effects
+				(font
+					(size 1.27 1.27)
+				)
+			)
+		)
+		(pin "2"
+		)
+		(pin "4"
+		)
+		(pin "1"
+		)
+		(pin "3"
+		)
+		(instances
+			(project "BILLEE_Science_Control_Module_V1"
+				(path "/0ccdd54c-cb66-4dbe-ac7e-21982bafb0a6/431a2b87-8d6b-4f12-9148-b0247a47a425"
+					(reference "U67")
+					(unit 1)
+				)
+			)
+		)
+	)
+	(symbol
 		(lib_id "scm_lib:Teyleten_Relay")
 		(at 251.46 82.55 0)
@@
 	)
 	(symbol
-		(lib_name "Roboclaw2x7A_1")
 		(lib_id "scm_lib:Roboclaw2x7A")
 		(at 138.43 78.74 0)
